Commit message: Enhance Gazebo textures and integrate strict sequence AprilTag tracking
- Fixed hardcoded absolute texture paths in SDF worlds via model URIs.
- Registered materials/ directory in CMakeLists.txt for portability.
- Repositioned mini_r1 coordinates to spawn centrally on base tile.
- Switched ArUco detector dictionary to DICT_APRILTAG_36h11.
- Implemented strict ArUco sequence tracking [2, 1, 3, 4, 5] logic in nav controller.
- Integrated dynamic distance-based execution threshold (<= 1.0m) preserving LiDAR constraints.

File: src/gazebo_gefier_r1-main/mini_r1_v1_description/urdf/robot_core.xacro (robot description, xacro)
@@ -15,4 +15,10 @@
         </visual>
     </xacro:property>
+    <link name="base_footprint"/>
+    <joint name="base_footprint_joint" type="fixed">
+        <parent link="base_footprint"/>
+        <child link="base_link"/>
+        <origin xyz="0 0 0" rpy="0 0 0"/>
+    </joint>
     <link name="base_link">
         <inertial>
